File: cc1111dongle/cc1111dongle.sch (KiCad schematic (older format))
At the start: 65 parts, among them J1 USB-DEVICE, P1 EXPANSION, P2 BNC-CONN, P3 RESET_N, P4 DD, P5 DC, P6 3V3, P7 GND, T1 BALUN, U1 CC1111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

Commit message: finished layout first pass
Connections:
- net 3V3: now also P1.1; no longer P1.10
- net AMP_BYPASS_EN: now also U1.17 (P2_3); no longer U1.32 (P1_7)
- net GND: now also P1.10; no longer P1.1
- net P0_0: now also P1.7; no longer P1.2
- net P0_1: now also P1.6; no longer P1.3
- net P0_2: now also P1.5; no longer P1.4
- net P0_3: now also P1.4; no longer P1.5
- net P1_2: now also R11.2; no longer P1.6
- net P1_3: now also R12.2; no longer P1.7
- net RX_AMP_EN: now also U1.18 (P2_4); no longer U1.33 (P1_6)
- net P1_1: now reaches R5.2, U1.3 (P1_1)
- net P0_5: now reaches U1.13 (P0_5)
- net P0_5: now also P1.2
- net P0_4: now reaches U1.9 (P0_4)
- net P0_4: now also P1.3
- net P1_4: no longer names the net of U1.35 (P1_4)
- net P1_4: no longer P1.8
- net P1_5: no longer names the net of U1.34 (P1_5)
- net P1_5: no longer P1.9
- removed net P2_3: R11.2, U1.17 (P2_3)
- removed net P2_4: R12.2, U1.18 (P2_4)
- new net P1_6: P1.9, U1.33 (P1_6)
- new net P1_7: P1.8, U1.32 (P1_7)
Other:
- moved on the sheet: D2, D3, D4, R11, R12, R5

Commit message: RF switch decoupling caps
Parts:
- added C27, C28: 100nF, symbol C
Connections:
- net 3V3: now also C27.2, C28.2
- net GND: now also C27.1, C28.1
Changed lines of the file:
@@
-EESchema Schematic File Version 2  date Sun Dec  9 21:56:22 2012
+EESchema Schematic File Version 2  date Mon Dec 10 16:58:36 2012
 LIBS:power
 LIBS:device
@@
 NoConn ~ 4850 3050
 NoConn ~ 4750 3050
+$Comp
+L C C27
+U 1 1 50C67AAE
+P 13850 3250
+F 0 "C27" H 13900 3350 50  0000 L CNN
+F 1 "100nF" H 13900 3150 50  0000 L CNN
+F 4 "Murata" H 13850 3250 60  0001 C CNN "Manufacturer"
+F 5 "GRM155R61A104KA01D" H 13850 3250 60  0001 C CNN "Part Number"
+F 6 "CAP CER 0.1UF 10V 10% X5R 0402" H 13850 3250 60  0001 C CNN "Description"
+	1    13850 3250
+	-1   0    0    1
+$EndComp
+$Comp
+L 3V3 #PWR065
+U 1 1 50C67AB4
+P 13850 2950
+F 0 "#PWR065" H 13850 3050 40  0001 C CNN
+F 1 "3V3" V 13850 3075 40  0000 C CNN
+	1    13850 2950
+	1    0    0    -1
+$EndComp
+$Comp
+L 3V3 #PWR066
+U 1 1 50C67ABA
+P 14200 2950
+F 0 "#PWR066" H 14200 3050 40  0001 C CNN
+F 1 "3V3" V 14200 3075 40  0000 C CNN
+	1    14200 2950
+	1    0    0    -1
+$EndComp
+$Comp
+L C C28
+U 1 1 50C67AC3
+P 14200 3250
+F 0 "C28" H 14250 3350 50  0000 L CNN
+F 1 "100nF" H 14250 3150 50  0000 L CNN
+F 4 "Murata" H 14200 3250 60  0001 C CNN "Manufacturer"
+F 5 "GRM155R61A104KA01D" H 14200 3250 60  0001 C CNN "Part Number"
+F 6 "CAP CER 0.1UF 10V 10% X5R 0402" H 14200 3250 60  0001 C CNN "Description"
+	1    14200 3250
+	-1   0    0    1
+$EndComp
+$Comp
+L GND #PWR067
+U 1 1 50C67AD5
+P 13850 3550
+F 0 "#PWR067" H 13850 3550 30  0001 C CNN
+F 1 "GND" H 13850 3480 30  0001 C CNN
+	1    13850 3550
+	1    0    0    -1
+$EndComp
+$Comp
+L GND #PWR068
+U 1 1 50C67AE2
+P 14200 3550
+F 0 "#PWR068" H 14200 3550 30  0001 C CNN
+F 1 "GND" H 14200 3480 30  0001 C CNN
+	1    14200 3550
+	1    0    0    -1
+$EndComp
+Wire Wire Line
+	14200 3050 14200 2950
+Wire Wire Line
+	13850 2950 13850 3050
+Wire Wire Line
+	13850 3450 13850 3550
+Wire Wire Line
+	14200 3450 14200 3550
 $EndSCHEMATC

Commit message: 11 jan 2013 update
Parts:
- C9: Part Number UMK105CG2R2CW-F -> UMK105CG2R2CV-F
Changed lines of the file:
@@
-EESchema Schematic File Version 2  date Mon Dec 10 16:58:36 2012
+EESchema Schematic File Version 2  date Sun Jan  6 11:43:45 2013
 LIBS:power
 LIBS:device
@@
 Sheet 1 1
 Title ""
-Date "10 dec 2012"
+Date "6 jan 2013"
 Rev ""
 Comp ""
@@
 F 1 "2p2" H 7750 4650 50  0000 L CNN
 F 4 "Taiyo Yuden" H 7700 4750 60  0001 C CNN "Manufacturer"
-F 5 "UMK105CG2R2CW-F" H 7700 4750 60  0001 C CNN "Part Number"
+F 5 "UMK105CG2R2CV-F" H 7700 4750 60  0001 C CNN "Part Number"
 F 6 "CAP CER 2.2PF 50V NP0 0402" H 7700 4750 60  0001 C CNN "Description"
 	1    7700 4750
